Commit message: changed youbot urdf

File: cleaner_alpha/robots/youbot.urdf.xacro (robot description, xacro)
@@ -48,6 +48,6 @@
   </xacro:youbot_gripper>
   <!-- camera at the gripper -->
-  <xacro:asus_xtion_camera name="${camera_name}" parent="${arm_name}_link_5" tilt="0.0" >
-    <origin xyz="0.035 0 0.005" rpy="0 ${M_PI/2.0} 0" />
+  <xacro:asus_xtion_camera name="${camera_name}" parent="${arm_name}_link_5" tilt="-0.15" >
+    <origin xyz="0.035 0 0.045" rpy="0 ${M_PI/2.0} 0" />
   </xacro:asus_xtion_camera>
   <link name="camera_link" />

Commit message: changed camera position and controls

File: cleaner_alpha/robots/youbot.urdf.xacro (robot description, xacro)
@@ -49,5 +49,5 @@
   <!-- camera at the gripper -->
   <xacro:asus_xtion_camera name="${camera_name}" parent="${arm_name}_link_5" tilt="-0.15" >
-    <origin xyz="0.035 0 0.045" rpy="0 ${M_PI/2.0} 0" />
+    <origin xyz="0.035 0 0.045" rpy="0 ${M_PI/2.0} ${M_PI}" />
   </xacro:asus_xtion_camera>
   <link name="camera_link" />

Commit message: fixed camera position...just a youbot sync

File: cleaner_alpha/robots/youbot.urdf.xacro (robot description, xacro)
@@ -49,5 +49,5 @@
   <!-- camera at the gripper -->
   <xacro:asus_xtion_camera name="${camera_name}" parent="${arm_name}_link_5" tilt="-0.15" >
-    <origin xyz="0.035 0 0.045" rpy="0 ${M_PI/2.0} ${M_PI}" />
+    <origin xyz="-0.035 0 0.045" rpy="0 ${M_PI/2.0} ${M_PI}" />
   </xacro:asus_xtion_camera>
   <link name="camera_link" />

Commit message: changed psoition control to not use the trajectory generator and some testing changes

File: cleaner_alpha/robots/youbot.urdf.xacro (robot description, xacro)
@@ -49,5 +49,5 @@
   <!-- camera at the gripper -->
   <xacro:asus_xtion_camera name="${camera_name}" parent="${arm_name}_link_5" tilt="-0.15" >
-    <origin xyz="-0.035 0 0.045" rpy="0 ${M_PI/2.0} ${M_PI}" />
+    <origin xyz="-0.02 0 0.045" rpy="0 ${M_PI/2.0} ${M_PI}" />
   </xacro:asus_xtion_camera>
   <link name="camera_link" />
